File: electrical/gameboy_rev_A/gameboy_rev_A.kicad_sch (KiCad schematic)
At the start: 8 parts, among them SW1 SW_SPST, U1 ESP32-WROOM-32D, U3 MAX98357, U4 MP2315 Buck

Commit message: send it
Parts:
- removed BT1: 3.7 V, symbol Device:Battery_Cell
- removed SW1: SW_SPST, symbol Switch:SW_SPST
- removed U4: MP2315 Buck, symbol gameboy_lib:MP2315_Mini_Adjustable_DC-DC_Step-Down_Module
Other:
- added sheet power_circuit (power_board.kicad_sch)

Commit message: okay
Parts:
- removed DS1: 3.5in SPI Display Module, symbol gameboy_lib:3.5in_SPI_Module_MSP3520
- removed LS1: Speaker, symbol Device:Speaker
- removed R1: 680k, symbol Device:R_US
- removed U3: MAX98357, symbol gameboy_lib:MAX98357A
Other:
- added sheet audio_circuit (audio_circuit.kicad_sch)
- added sheet display_memory circuit (display_circuit.kicad_sch)
- added sheet input_circuit (input_circuit.kicad_sch)
- note removed: "Range Supply Voltage 2.5 - 5.5"
- note removed: "SD_MODE Voltage Divider, Internal pulldown 100k, bias between 0.17-0.77 v for dual channel speaker R_1 = (3.3 v - 0.465 v)/(.465v/100k) = 609k ~ 680k"

Commit message: beautiful flowchart
Parts:
- removed U1: ESP32-WROOM-32D, RF_Module:ESP32-WROOM-32D, symbol RF_Module:ESP32-WROOM-32D
Other:
- note added: "18650 Battery"
- note added: "3.3v Regulator"
- note added: "Buttons"
- note added: "DAC + Audio Amp Circuit"
- note added: "ESP32"
- note added: "LCD Display SD Card Slot"
- note added: "USB-C Charging"
- note removed: "disable regulators via GPIO if in deep sleep removing boost converter, 3.3 v is fine for backlight LED"
