File: electrical/gameboy_rev_A/power_board.kicad_sch (KiCad schematic)
At the start: 3 parts, among them SW1 SW_SPST, U4 MP2315 Buck

Commit message: beautiful flowchart
Other:
- note added: "disable regulators via GPIO if in deep sleep removing boost converter, 3.3 v is fine for backlight LED"
Changed lines of the file:
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@@
 	(generator_version "9.0")
 	(paper "A5")
+	(text "disable regulators via GPIO if in deep sleep\nremoving boost converter, 3.3 v is fine for backlight LED\n"
+		(exclude_from_sim no)
+		(at 134.874 49.276 0)
+		(effects
+			(font
+				(size 1.27 1.27)
+			)
+		)
+	)
 	(junction
 		(at 102.87 63.5)
