File: electrical/gameboy_rev_A/input_circuit.kicad_sch (KiCad schematic)
At the start: 0 parts

Commit message: dpad added
Parts:
- added SW2: ~, symbol gameboy_lib:5_Way_DPad_Switch_SMD_COM-26850
Connections:
- new net +3.3V: SW2.10, SW2.3, SW2.5, SW2.8
- new net GND: SW2.4, SW2.9
